File: pcb/right/keyboard_pcb.kicad_pcb (KiCad board)
At the start: 2 copper layers, 138.8 x 89.9 mm, 36 parts, among them J2 USB_C_Receptacle_USB2.0_16P, K00 KEYSW, K01 KEYSW, K02 KEYSW, K03 KEYSW, K04 KEYSW, K05 KEYSW, K10 KEYSW, K11 KEYSW, K12 KEYSW, K13 KEYSW, K14 KEYSW, K15 KEYSW, K20 KEYSW, K21 KEYSW, K22 KEYSW, K23 KEYSW, K24 KEYSW, K25 KEYSW, K30 KEYSW, K31 KEYSW, K32 KEYSW, U2 Pico

Commit message: Update right side
Connections:
- J2 pad A6: tx -> rx
- J2 pad A7: rx -> tx
- J2 pad B6: tx -> rx
- J2 pad B7: rx -> tx
Routing:
- net rx: track 59.1 -> 60.4 mm
- net tx: track 63.0 -> 61.7 mm, vias 0 -> 2
Changed lines of the file:
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@@
 			(drillshape 0)
 			(scaleselection 1)
-			(outputdirectory "../Fabrication/")
+			(outputdirectory "../fabrication/right/")
 		)
 	)
@@
 		)
 		(pad "" np_thru_hole circle
-			(at 5.000001 -3.75 355)
+			(at 5.000003 -3.75 355)
 			(size 3 3)
 			(drill 3)
@@
 			(size 0.3 1.16)
 			(layers "F.Cu" "F.Paste" "F.Mask")
-			(net 24 "tx")
+			(net 23 "rx")
 			(pinfunction "D+")
 			(pintype "bidirectional")
@@
 			(size 0.3 1.16)
 			(layers "F.Cu" "F.Paste" "F.Mask")
-			(net 23 "rx")
+			(net 24 "tx")
 			(pinfunction "D-")
 			(pintype "bidirectional")
@@
 			(size 0.3 1.16)
 			(layers "F.Cu" "F.Paste" "F.Mask")
-			(net 24 "tx")
+			(net 23 "rx")
 			(pinfunction "D+")
 			(pintype "bidirectional")
@@
 			(size 0.3 1.16)
 			(layers "F.Cu" "F.Paste" "F.Mask")
-			(net 23 "rx")
+			(net 24 "tx")
 			(pinfunction "D-")
 			(pintype "bidirectional")
@@
 		)
 		(fp_line
-			(start -2 -4.749999)
+			(start -2 -4.749998)
 			(end -4.5 -4.75)
 			(stroke
@@
 	)
 	(segment
-		(start 72.45 109.25)
-		(end 73.31 109.25)
+		(start 75.2 60.6712)
+		(end 74.6 60.0712)
 		(width 0.25)
 		(layer "F.Cu")
@@
 	)
 	(segment
-		(start 72.2 109)
-		(end 72.45 109.25)
+		(start 74.6 109.16)
+		(end 74.6 109.4)
 		(width 0.25)
 		(layer "F.Cu")
@@
 	)
 	(segment
-		(start 73.31 108.25)
-		(end 72.43 108.25)
+		(start 73.31 108.75)
+		(end 74.19 108.75)
 		(width 0.25)
 		(layer "F.Cu")
@@
 	)
 	(segment
-		(start 74.15 108.25)
-		(end 73.31 108.25)
+		(start 74.25 109.75)
+		(end 73.31 109.75)
+		(width 0.25)
+		(layer "F.Cu")
+		(net 23)
+	)
+	(segment
+		(start 75.2 107.836396)
+		(end 75.2 60.6712)
 		(width 0.25)
 		(layer "F.Cu")
@@
 	)
 	(segment
-		(start 74.6 60.0712)
-		(end 74.6 107.8)
+		(start 74.286396 108.75)
+		(end 73.31 108.75)
 		(width 0.25)
 		(layer "F.Cu")
@@
 	)
 	(segment
-		(start 72.43 108.25)
-		(end 72.2 108.48)
+		(start 74.6 109.4)
+		(end 74.25 109.75)
 		(width 0.25)
 		(layer "F.Cu")
@@
 	)
 	(segment
-		(start 72.2 108.48)
-		(end 72.2 109)
+		(start 75.2 107.836396)
+		(end 74.286396 108.75)
 		(width 0.25)
 		(layer "F.Cu")
@@
 	)
 	(segment
-		(start 74.6 107.8)
-		(end 74.15 108.25)
+		(start 74.19 108.75)
+		(end 74.6 109.16)
 		(width 0.25)
 		(layer "F.Cu")
@@
 	)
 	(segment
-		(start 74.6 109.16)
-		(end 74.6 109.4)
+		(start 73.2438 56.175)
+		(end 73.25 56.175)
 		(width 0.25)
 		(layer "F.Cu")
@@
 	)
 	(segment
-		(start 73.31 108.75)
-		(end 74.19 108.75)
+		(start 72.45 109.25)
+		(end 73.31 109.25)
 		(width 0.25)
 		(layer "F.Cu")
@@
 	)
 	(segment
-		(start 75.2 58.1312)
-		(end 75.2 107.836396)
+		(start 72.2 109)
+		(end 72.45 109.25)
 		(width 0.25)
 		(layer "F.Cu")
@@
 	)
 	(segment
-		(start 74.25 109.75)
-		(end 73.31 109.75)
+		(start 73.31 108.25)
+		(end 72.43 108.25)
+		(width 0.25)
+		(layer "F.Cu")
+		(net 24)
+	)
+	(segment
+		(start 74.6 61.925)
+		(end 74.6 107.8)
 		(width 0.25)
 		(layer "F.Cu")
@@
 	(segment
 		(start 69.6468 52.578)
-		(end 75.2 58.1312)
+		(end 73.2438 56.175)
 		(width 0.25)
 		(layer "F.Cu")
@@
 	)
 	(segment
-		(start 74.286396 108.75)
-		(end 73.31 108.75)
+		(start 74.15 108.25)
+		(end 73.31 108.25)
 		(width 0.25)
 		(layer "F.Cu")
@@
 	)
 	(segment
-		(start 74.6 109.4)
-		(end 74.25 109.75)
+		(start 72.43 108.25)
+		(end 72.2 108.48)
 		(width 0.25)
 		(layer "F.Cu")
@@
 	)
 	(segment
-		(start 75.2 107.836396)
-		(end 74.286396 108.75)
+		(start 72.2 108.48)
+		(end 72.2 109)
 		(width 0.25)
 		(layer "F.Cu")
@@
 	)
 	(segment
-		(start 74.19 108.75)
-		(end 74.6 109.16)
+		(start 74.6 107.8)
+		(end 74.15 108.25)
+		(width 0.25)
+		(layer "F.Cu")
+		(net 24)
+	)
+	(segment
+		(start 73.25 60.575)
+		(end 74.6 61.925)
 		(width 0.25)
 		(layer "F.Cu")
 		(net 24)
 	)
+	(via
+		(at 73.25 56.175)
+		(size 0.6)
+		(drill 0.3)
+		(layers "F.Cu" "B.Cu")
+		(net 24)
+	)
+	(via
+		(at 73.25 60.575)
+		(size 0.6)
+		(drill 0.3)
+		(layers "F.Cu" "B.Cu")
+		(free yes)
+		(net 24)
+	)
+	(segment
+		(start 73.25 60.575)
+		(end 73.25 56.175)
+		(width 0.25)
+		(layer "B.Cu")
+		(net 24)
+	)
